File: kicad/clock.kicad_pcb (KiCad board)
At the start: 4 copper layers, 87 x 38 mm, 56 parts, among them P1 CONN_01X03, SW1 SWITCH_MIN, SW2 SWITCH_HR, U1 74LS90, U10 74LS247, U11 74LS73, U2 74LS90, U3 MAX6817, U4 74LS90, U5 74LS247, U6 74LS90, U7 74LS00, U8 74LS247, U9 74LS163

Commit message: More routing improvements
Routing:
- net /hoi1: track 51.8 -> 50.0 mm
- net /mti0: track 39.3 -> 38.2 mm

Commit message: Add BoM, update component info, use 150Ohm current limiting resistors, update layout respectively
Parts:
- R1, R10, R11, R14, R15, R16, R17, R18, R19, R2, R20, R21, R22, R23, R24, R25, R26, R27, R3, R4, R5, R6, R7, R8, R9: value 220Ω -> 150Ω
- turned R4 to 270 degrees
Connections:
- R4 pad 1: Net-(R4-Pad1) -> /ht
- R4 pad 2: /ht -> Net-(R4-Pad2)
- S1 pad 4: Net-(R4-Pad1) -> Net-(R4-Pad2)
Routing:
- net Net-(R4-Pad2): track 0.00 -> 3.29 mm
- net Net-(R4-Pad1): track 3.29 -> 0.00 mm
